Commit message: add effort and velocity  controller for joint_1 and joint_2

File: models/urdf/s500_uam_arm_velocity.urdf.xacro (robot description, xacro)
@@ -54,5 +54,5 @@
     <child link="link_1"/>
     <axis xyz="0 1 0"/>
-    <limit lower="-1.57" upper="1.57" effort="10" velocity="1"/>
+    <limit lower="-1.57" upper="1.57" effort="2" velocity="1"/>
   </joint>
   <!-- Link 2 -->
@@ -82,5 +82,5 @@
     <child link="link_2"/>
     <axis xyz="0 1 0"/>
-    <limit lower="-1.57" upper="1.57" effort="10" velocity="1"/>
+    <limit lower="-1.57" upper="1.57" effort="2" velocity="1"/>
   </joint>
   <!-- Link 3 (Gripper Left Finger) -->
@@ -110,5 +110,5 @@
     <child link="link_3"/>
     <axis xyz="0 1 0"/>
-    <limit lower="-1.57" upper="1.57" effort="10" velocity="1"/>
+    <limit lower="-1.57" upper="1.57" effort="2" velocity="1"/>
   </joint>
   <!-- Link 4 (Gripper Right Finger - mimic) -->
@@ -138,5 +138,5 @@
     <child link="link_4"/>
     <axis xyz="0 1 0"/>
-    <limit lower="-1.57" upper="1.57" effort="10" velocity="1"/>
+    <limit lower="-1.57" upper="1.57" effort="2" velocity="1"/>
   </joint>
   <!-- Transmissions for ros_control -->
@@ -144,9 +144,7 @@
     <type>transmission_interface/SimpleTransmission</type>
     <joint name="joint_1">
-      <hardwareInterface>hardware_interface/PositionJointInterface</hardwareInterface>
+      <hardwareInterface>hardware_interface/VelocityJointInterface</hardwareInterface>
     </joint>
     <actuator name="joint_1_motor">
-      <hardwareInterface>hardware_interface/PositionJointInterface</hardwareInterface>
-      <mechanicalReduction>1.0</mechanicalReduction>
     </actuator>
   </transmission>
@@ -154,9 +152,7 @@
     <type>transmission_interface/SimpleTransmission</type>
     <joint name="joint_2">
-      <hardwareInterface>hardware_interface/PositionJointInterface</hardwareInterface>
+      <hardwareInterface>hardware_interface/VelocityJointInterface</hardwareInterface>
     </joint>
     <actuator name="joint_2_motor">
-      <hardwareInterface>hardware_interface/PositionJointInterface</hardwareInterface>
-      <mechanicalReduction>1.0</mechanicalReduction>
     </actuator>
   </transmission>
@@ -167,6 +163,4 @@
     </joint>
     <actuator name="joint_3_motor">
-      <hardwareInterface>hardware_interface/PositionJointInterface</hardwareInterface>
-      <mechanicalReduction>1.0</mechanicalReduction>
     </actuator>
   </transmission>
@@ -177,6 +171,4 @@
     </joint>
     <actuator name="joint_4_motor">
-      <hardwareInterface>hardware_interface/PositionJointInterface</hardwareInterface>
-      <mechanicalReduction>1.0</mechanicalReduction>
     </actuator>
   </transmission>

File: models/urdf/s500_uam_simple_0717.urdf (robot description, URDF)
Before this commit: robot s500_uam, 10 links, 9 joints
Joints:
- joint joint_1: limit lower=-1.5 upper=1.5 effort=1 velocity=3 -> lower=-1.5 upper=1.5 effort=1 velocity=1
- joint joint_2: limit lower=-1.5 upper=1.5 effort=1 velocity=3 -> lower=-1.0 upper=1.0 effort=1 velocity=1
