Commit message: update s500 simple urdf file

File: models/urdf/s500_simple.urdf (robot description, URDF)
Before this commit: robot s500_quadrotor, 5 links, 4 joints
Links:
- link rotor_1: mass 0.010198 -> 0.01
- link rotor_2: mass 0.010198 -> 0.01
- link rotor_3: mass 0.010198 -> 0.01
- link rotor_4: mass 0.010198 -> 0.01
Joints:
- joint rotor_joint_1: origin xyz=0.171 0.171 0.045 rpy=0 0 0 -> xyz=0.171 0.171 0.07 rpy=0 0 0
- joint rotor_joint_2: origin xyz=-0.171 0.171 0.045 rpy=0 0 0 -> xyz=-0.171 0.171 0.07 rpy=0 0 0
- joint rotor_joint_3: origin xyz=-0.171 -0.171 0.045 rpy=0 0 0 -> xyz=-0.171 -0.171 0.07 rpy=0 0 0
- joint rotor_joint_4: origin xyz=0.1701 -0.1701 0.0603 rpy=0 0 0 -> xyz=0.171 -0.171 0.07 rpy=0 0 0
