Commit message: update urdf files

File: models/urdf/s500_uam_arm_effort.urdf (robot description, URDF)
Before this commit: robot s500_uam_arm, 7 links, 6 joints
Joints:
- joint joint_3: type revolute -> fixed
- joint joint_4: type revolute -> fixed

File: models/urdf/s500_uam_arm_effort.urdf.xacro (robot description, xacro)
@@ -139,4 +139,34 @@
     <axis xyz="0 1 0"/>
     <limit lower="-1.57" upper="1.57" effort="2" velocity="1"/>
+  </joint>
+  <!-- Gripper -->
+  <link name="gripper_link">
+    <visual>
+      <origin xyz="0 0 0" rpy="0 0 0"/>
+      <geometry>
+        <box size="0.01 0.01 0.01"/>
+      </geometry>
+      <material name="red">
+        <color rgba="1 0 0 1"/>
+      </material>
+    </visual>
+    <collision>
+      <origin xyz="0 0 0" rpy="0 0 0"/>
+      <geometry>
+        <box size="0.01 0.01 0.01"/>
+      </geometry>
+    </collision>
+    <inertial>
+      <origin xyz="0.024422 -0.000991 -0.039818" rpy="0 0 0"/>
+      <mass value="0.001"/>
+      <inertia ixx="1.1294e-05" ixy="2.4212e-09" ixz="4.0228e-06"
+               iyy="1.352e-05" iyz="-4.1022e-09" izz="2.6966e-06"/>
+    </inertial>
+  </link>
+  <!-- Gripper Joint -->
+  <joint name="gripper_joint" type="fixed">
+    <parent link="link_2"/>
+    <child link="gripper_link"/>
+    <origin xyz="0 0 -0.14" rpy="0 0 0"/>
   </joint>
   <!-- Transmissions for ros_control -->

File: models/urdf/s500_uam_arm_velocity.urdf.xacro (robot description, xacro)
@@ -139,4 +139,34 @@
     <axis xyz="0 1 0"/>
     <limit lower="-1.57" upper="1.57" effort="2" velocity="1"/>
+  </joint>
+  <!-- Gripper -->
+  <link name="gripper_link">
+    <visual>
+      <origin xyz="0 0 0" rpy="0 0 0"/>
+      <geometry>
+        <box size="0.01 0.01 0.01"/>
+      </geometry>
+      <material name="red">
+        <color rgba="1 0 0 1"/>
+      </material>
+    </visual>
+    <collision>
+      <origin xyz="0 0 0" rpy="0 0 0"/>
+      <geometry>
+        <box size="0.01 0.01 0.01"/>
+      </geometry>
+    </collision>
+    <inertial>
+      <origin xyz="0.024422 -0.000991 -0.039818" rpy="0 0 0"/>
+      <mass value="0.001"/>
+      <inertia ixx="1.1294e-05" ixy="2.4212e-09" ixz="4.0228e-06"
+               iyy="1.352e-05" iyz="-4.1022e-09" izz="2.6966e-06"/>
+    </inertial>
+  </link>
+  <!-- Gripper Joint -->
+  <joint name="gripper_joint" type="fixed">
+    <parent link="link_2"/>
+    <child link="gripper_link"/>
+    <origin xyz="0 0 -0.14" rpy="0 0 0"/>
   </joint>
   <!-- Transmissions for ros_control -->

Commit message: update target weight to 200g

File: models/urdf/s500_uam_arm_effort.urdf (robot description, URDF)
Before this commit: robot s500_uam_arm, 7 links, 6 joints
Links:
- link gripper_link: geometry visual box size=0.01 0.01 0.01
- link link_1: mass 0.056776 -> 0.095; geometry collision mesh filename=package://example-robot-data/robots/s500_description/s500_u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; visual mesh filename=package://example-robot-data/robots/s500_description/s500_u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
- link link_2: mass 0.065663 -> 0.082; geometry collision mesh filename=package://example-robot-data/robots/s500_description/s500_u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; visual mesh filename=package://example-robot-data/robots/s500_description/s500_u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
- link link_3: mass 0.012158 -> 0.012; geometry collision mesh filename=package://example-robot-data/robots/s500_description/s500_u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; visual mesh filename=package://example-robot-data/robots/s500_description/s500_u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
- link link_4: mass 0.012587 -> 0.012; geometry collision mesh filename=package://example-robot-data/robots/s500_description/s500_u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; visual mesh filename=package://example-robot-data/robots/s500_description/s500_u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
Joints:
- joint joint_1: limit lower=-1.57 upper=1.57 effort=2 velocity=1 -> lower=-2 upper=2 effort=10 velocity=20; origin xyz=0.0007 0 -0.00275 rpy=0 0 0 -> xyz=0.0007 0 -0.07275 rpy=0 0 0
- joint joint_2: limit lower=-1.57 upper=1.57 effort=2 velocity=1 -> lower=-2 upper=2 effort=10 velocity=20
- joint joint_3: limit lower=-1.57 upper=1.57 effort=2 velocity=1 -> lower=-1.57 upper=0 effort=10 velocity=1; origin xyz=-0.011 0 -0.08225 rpy=0 0.23432 -3.14159 -> xyz=-0.011 0 -0.08225 rpy=0 0.23432 3.1416
- joint joint_4: limit lower=-1.57 upper=1.57 effort=2 velocity=1 -> lower=0 upper=1.57 effort=10 velocity=1

File: models/urdf/s500_uam_arm_effort.urdf.xacro (robot description, xacro)
@@ -32,7 +32,7 @@
     <inertial>
       <origin xyz="-0 -0.000196 -0.076809" rpy="0 0 0"/>
-      <mass value="0.056776"/>
-      <inertia ixx="1.5689e-05" ixy="-1.0155e-16" ixz="-5.2428e-15"
-               iyy="1.3617e-05" iyz="-1.6017e-09" izz="8.7857e-06"/>
+      <mass value="0.095"/>
+      <inertia ixx="5.8e-05" ixy="0" ixz="0"
+               iyy="5.1e-05" iyz="0" izz="1.8e-05"/>
     </inertial>
     <visual>
@@ -54,5 +54,9 @@
     <child link="link_1"/>
     <axis xyz="0 1 0"/>
-    <limit lower="-1.57" upper="1.57" effort="2" velocity="1"/>
+    <limit lower="-1.57" upper="1.57" effort="1" velocity="1"/>
+    <dynamics>
+      <damping>0.05</damping>
+      <friction>0.1</friction>
+    </dynamics>
   </joint>
   <!-- Link 2 -->
@@ -60,7 +64,7 @@
     <inertial>
       <origin xyz="0.000575 0.000247 -0.072261" rpy="0 0 0"/>
-      <mass value="0.065663"/>
-      <inertia ixx="1.3006e-05" ixy="2.5553e-07" ixz="4.4082e-09"
-               iyy="1.4985e-05" iyz="-6.0777e-07" izz="1.6054e-05"/>
+      <mass value="0.082"/>
+      <inertia ixx="4.3e-05" ixy="0" ixz="0"
+               iyy="4.1e-05" iyz="0" izz="2.6e-05"/>
     </inertial>
     <visual>
@@ -82,5 +86,9 @@
     <child link="link_2"/>
     <axis xyz="0 1 0"/>
-    <limit lower="-1.57" upper="1.57" effort="2" velocity="1"/>
+    <limit lower="-1.57" upper="1.57" effort="1" velocity="1"/>
+    <dynamics>
+      <damping>0.05</damping>
+      <friction>0.1</friction>
+    </dynamics>
   </joint>
   <!-- Link 3 (Gripper Left Finger) -->
@@ -88,7 +96,7 @@
     <inertial>
       <origin xyz="0.025274 0.000991 -0.041284" rpy="0 0 0"/>
-      <mass value="0.012158"/>
-      <inertia ixx="1.0667e-05" ixy="-2.5213e-09" ixz="3.6553e-06"
-               iyy="1.2675e-05" iyz="4.2721e-09" izz="2.4775e-06"/>
+      <mass value="0.012"/>
+      <inertia ixx="1.0e-05" ixy="0" ixz="0"
+               iyy="1.0e-05" iyz="0" izz="2.0e-06"/>
     </inertial>
     <visual>
@@ -110,5 +118,5 @@
     <child link="link_3"/>
     <axis xyz="0 1 0"/>
-    <limit lower="-1.57" upper="1.57" effort="2" velocity="1"/>
+    <limit lower="-1.57" upper="1.57" effort="0.5" velocity="0.5"/>
   </joint>
   <!-- Link 4 (Gripper Right Finger - mimic) -->
@@ -116,7 +124,7 @@
     <inertial>
       <origin xyz="0.024422 -0.000991 -0.039818" rpy="0 0 0"/>
-      <mass value="0.012587"/>
-      <inertia ixx="1.1294e-05" ixy="2.4212e-09" ixz="4.0228e-06"
-               iyy="1.352e-05" iyz="-4.1022e-09" izz="2.6966e-06"/>
+      <mass value="0.012"/>
+      <inertia ixx="1.0e-05" ixy="0" ixz="0"
+               iyy="1.0e-05" iyz="0" izz="2.0e-06"/>
     </inertial>
     <visual>
@@ -138,8 +146,8 @@
     <child link="link_4"/>
     <axis xyz="0 1 0"/>
-    <limit lower="-1.57" upper="1.57" effort="2" velocity="1"/>
+    <limit lower="-1.57" upper="1.57" effort="1.0" velocity="0.5"/>
   </joint>
   <!-- Gripper -->
-  <link name="gripper_link">
+  <!-- <link name="gripper_link">
     <visual>
       <origin xyz="0 0 0" rpy="0 0 0"/>
@@ -164,10 +172,9 @@
     </inertial>
   </link>
-  <!-- Gripper Joint -->
   <joint name="gripper_joint" type="fixed">
     <parent link="link_2"/>
     <child link="gripper_link"/>
     <origin xyz="0 0 -0.14" rpy="0 0 0"/>
-  </joint>
+  </joint> -->
   <!-- Transmissions for ros_control -->
   <transmission name="joint_1_trans">
@@ -202,7 +209,7 @@
     <type>transmission_interface/SimpleTransmission</type>
     <joint name="joint_3">
-      <hardwareInterface>hardware_interface/PositionJointInterface</hardwareInterface>
-      <!-- <hardwareInterface>hardware_interface/VelocityJointInterface</hardwareInterface>
-      <hardwareInterface>hardware_interface/EffortJointInterface</hardwareInterface> -->
+      <!-- <hardwareInterface>hardware_interface/PositionJointInterface</hardwareInterface> -->
+      <!-- <hardwareInterface>hardware_interface/VelocityJointInterface</hardwareInterface> -->
+      <hardwareInterface>hardware_interface/EffortJointInterface</hardwareInterface>
     </joint>
     <actuator name="joint_3_motor">
@@ -216,7 +223,7 @@
     <type>transmission_interface/SimpleTransmission</type>
     <joint name="joint_4">
-      <hardwareInterface>hardware_interface/PositionJointInterface</hardwareInterface>
-      <!-- <hardwareInterface>hardware_interface/VelocityJointInterface</hardwareInterface>
-      <hardwareInterface>hardware_interface/EffortJointInterface</hardwareInterface> -->
+      <!-- <hardwareInterface>hardware_interface/PositionJointInterface</hardwareInterface> -->
+      <!-- <hardwareInterface>hardware_interface/VelocityJointInterface</hardwareInterface> -->
+      <hardwareInterface>hardware_interface/EffortJointInterface</hardwareInterface>
     </joint>
     <actuator name="joint_4_motor">
@@ -231,4 +238,5 @@
       <robotNamespace>/s500_uam</robotNamespace>
       <controlPeriod>0.001</controlPeriod>
+      <updateRate>1000</updateRate>
       <robotParam>/s500_uam/robot_description</robotParam>
       <legacyModeNS>true</legacyModeNS>

File: models/urdf/s500_uam_arm_position.urdf.xacro (robot description, xacro)
@@ -32,7 +32,7 @@
     <inertial>
       <origin xyz="-0 -0.000196 -0.076809" rpy="0 0 0"/>
-      <mass value="0.056776"/>
-      <inertia ixx="1.5689e-05" ixy="-1.0155e-16" ixz="-5.2428e-15"
-               iyy="1.3617e-05" iyz="-1.6017e-09" izz="8.7857e-06"/>
+      <mass value="0.095"/>
+      <inertia ixx="5.8e-05" ixy="0" ixz="0"
+               iyy="5.1e-05" iyz="0" izz="1.8e-05"/>
     </inertial>
     <visual>
@@ -54,5 +54,9 @@
     <child link="link_1"/>
     <axis xyz="0 1 0"/>
-    <limit lower="-1.57" upper="1.57" effort="2" velocity="1"/>
+    <limit lower="-1.57" upper="1.57" effort="1" velocity="1"/>
+    <dynamics>
+      <damping>0.05</damping>
+      <friction>0.1</friction>
+    </dynamics>
   </joint>
   <!-- Link 2 -->
@@ -60,7 +64,7 @@
     <inertial>
       <origin xyz="0.000575 0.000247 -0.072261" rpy="0 0 0"/>
-      <mass value="0.065663"/>
-      <inertia ixx="1.3006e-05" ixy="2.5553e-07" ixz="4.4082e-09"
-               iyy="1.4985e-05" iyz="-6.0777e-07" izz="1.6054e-05"/>
+      <mass value="0.082"/>
+      <inertia ixx="4.3e-05" ixy="0" ixz="0"
+               iyy="4.1e-05" iyz="0" izz="2.6e-05"/>
     </inertial>
     <visual>
@@ -82,5 +86,9 @@
     <child link="link_2"/>
     <axis xyz="0 1 0"/>
-    <limit lower="-1.57" upper="1.57" effort="2" velocity="1"/>
+    <limit lower="-1.57" upper="1.57" effort="1" velocity="1"/>
+    <dynamics>
+      <damping>0.05</damping>
+      <friction>0.1</friction>
+    </dynamics>
   </joint>
   <!-- Link 3 (Gripper Left Finger) -->
@@ -88,7 +96,7 @@
     <inertial>
       <origin xyz="0.025274 0.000991 -0.041284" rpy="0 0 0"/>
-      <mass value="0.012158"/>
-      <inertia ixx="1.0667e-05" ixy="-2.5213e-09" ixz="3.6553e-06"
-               iyy="1.2675e-05" iyz="4.2721e-09" izz="2.4775e-06"/>
+      <mass value="0.012"/>
+      <inertia ixx="1.0e-05" ixy="0" ixz="0"
+               iyy="1.0e-05" iyz="0" izz="2.0e-06"/>
     </inertial>
     <visual>
@@ -110,5 +118,5 @@
     <child link="link_3"/>
     <axis xyz="0 1 0"/>
-    <limit lower="-1.57" upper="1.57" effort="2" velocity="1"/>
+    <limit lower="-1.57" upper="1.57" effort="0.5" velocity="0.5"/>
   </joint>
   <!-- Link 4 (Gripper Right Finger - mimic) -->
@@ -116,7 +124,7 @@
     <inertial>
       <origin xyz="0.024422 -0.000991 -0.039818" rpy="0 0 0"/>
-      <mass value="0.012587"/>
-      <inertia ixx="1.1294e-05" ixy="2.4212e-09" ixz="4.0228e-06"
-               iyy="1.352e-05" iyz="-4.1022e-09" izz="2.6966e-06"/>
+      <mass value="0.012"/>
+      <inertia ixx="1.0e-05" ixy="0" ixz="0"
+               iyy="1.0e-05" iyz="0" izz="2.0e-06"/>
     </inertial>
     <visual>
@@ -138,8 +146,8 @@
     <child link="link_4"/>
     <axis xyz="0 1 0"/>
-    <limit lower="-1.57" upper="1.57" effort="2" velocity="1"/>
+    <limit lower="-1.57" upper="1.57" effort="1.0" velocity="0.5"/>
   </joint>
   <!-- Gripper -->
-  <link name="gripper_link">
+  <!-- <link name="gripper_link">
     <visual>
       <origin xyz="0 0 0" rpy="0 0 0"/>
@@ -164,10 +172,9 @@
     </inertial>
   </link>
-  <!-- Gripper Joint -->
   <joint name="gripper_joint" type="fixed">
     <parent link="link_2"/>
     <child link="gripper_link"/>
     <origin xyz="0 0 -0.14" rpy="0 0 0"/>
-  </joint>
+  </joint> -->
   <!-- Transmissions for ros_control -->
   <transmission name="joint_1_trans">
@@ -177,4 +184,8 @@
     </joint>
     <actuator name="joint_1_motor">
+        <hardwareInterface>hardware_interface/PositionJointInterface</hardwareInterface>
+        <hardwareInterface>hardware_interface/VelocityJointInterface</hardwareInterface>
+        <hardwareInterface>hardware_interface/EffortJointInterface</hardwareInterface>
+        <mechanicalReduction>1.0</mechanicalReduction>
     </actuator>
   </transmission>
@@ -185,4 +196,8 @@
     </joint>
     <actuator name="joint_2_motor">
+        <hardwareInterface>hardware_interface/PositionJointInterface</hardwareInterface>
+        <hardwareInterface>hardware_interface/VelocityJointInterface</hardwareInterface>
+        <hardwareInterface>hardware_interface/EffortJointInterface</hardwareInterface>
+        <mechanicalReduction>1.0</mechanicalReduction>
     </actuator>
   </transmission>
@@ -207,4 +222,5 @@
       <robotNamespace>/s500_uam</robotNamespace>
       <controlPeriod>0.001</controlPeriod>
+      <updateRate>1000</updateRate>
       <robotParam>/s500_uam/robot_description</robotParam>
       <legacyModeNS>true</legacyModeNS>

File: models/urdf/s500_uam_simple.urdf (robot description, URDF)
Before this commit: robot s500_uam, 10 links, 9 joints
Links:
- link gripper_link: mass None -> 0.001
- link link_1: mass 0.056776 -> 0.095
- link link_2: mass 0.065663 -> 0.082
- link link_3: mass 0.012158 -> 0.012
- link link_4: mass 0.012587 -> 0.012
- link rotor_1: mass 0.010198 -> 0.01
- link rotor_2: mass 0.010198 -> 0.01
- link rotor_3: mass 0.010198 -> 0.01
- link rotor_4: mass 0.010198 -> 0.01
Joints:
- joint joint_1: limit lower=-1.5 upper=1.5 effort=1 velocity=3 -> lower=-2 upper=2 effort=2 velocity=10
- joint joint_2: limit lower=-1.5 upper=1.5 effort=1 velocity=3 -> lower=-2 upper=2 effort=2 velocity=10

File: models/urdf/s500_uam_simple_0717.urdf (robot description, URDF)
Before this commit: robot s500_uam, 10 links, 9 joints
Joints:
- joint joint_3: type fixed -> revolute
- joint joint_4: type fixed -> revolute
